File: GaussSpeedway.kicad_sch (KiCad schematic)
At the start: 47 parts, among them J1 Barrel_Jack_Switch, J2 JST PH, T1 LinearTouch4, T2 Conn_01x01, T3 LinearTouch4, U1 STM32F051C6Tx, U2 MCP1754S-3302xCB, U3 ZXBM5210-SP, U4 ZXBM5210-SP, U5 ZXBM5210-SP

Commit message: Updates for rev 3
- Expand planes and add vias under hbridge drivers for better thermal
dissipation
- Add some thermal dissipation planes on inductor pads
- Move guard rail current crossover to In2, further from cars and
closer to the balanced return current on the bottom layer
- Increase drive trace width from 0.3 to 0.45mm
- Increase mounting holes from 3.5mm to 3.7mm
Parts:
- H1, H2, H3, H4: footprint MountingHole:MountingHole_3.5mm -> MountingHole:MountingHole_3.7mm
Changed lines of the file:
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@@
       (effects (font (size 1.27 1.27)) (justify left))
     )
-    (property "Footprint" "MountingHole:MountingHole_3.5mm" (id 2) (at 21.59 44.45 0)
+    (property "Footprint" "MountingHole:MountingHole_3.7mm" (id 2) (at 21.59 44.45 0)
       (effects (font (size 1.27 1.27)) hide)
     )
@@
       (effects (font (size 1.27 1.27)) (justify left))
     )
-    (property "Footprint" "MountingHole:MountingHole_3.5mm" (id 2) (at 21.59 24.765 0)
+    (property "Footprint" "MountingHole:MountingHole_3.7mm" (id 2) (at 21.59 24.765 0)
       (effects (font (size 1.27 1.27)) hide)
     )
@@
       (effects (font (size 1.27 1.27)) (justify left))
     )
-    (property "Footprint" "MountingHole:MountingHole_3.5mm" (id 2) (at 21.59 38.735 0)
+    (property "Footprint" "MountingHole:MountingHole_3.7mm" (id 2) (at 21.59 38.735 0)
       (effects (font (size 1.27 1.27)) hide)
     )
@@
       (effects (font (size 1.27 1.27)) (justify left))
     )
-    (property "Footprint" "MountingHole:MountingHole_3.5mm" (id 2) (at 21.59 31.115 0)
+    (property "Footprint" "MountingHole:MountingHole_3.7mm" (id 2) (at 21.59 31.115 0)
       (effects (font (size 1.27 1.27)) hide)
     )
@@
     )
     (path "/8bdea5f6-7a53-427a-92b8-fd15994c2e8c"
-      (reference "H1") (unit 1) (value "MountingHole") (footprint "MountingHole:MountingHole_3.5mm")
+      (reference "H1") (unit 1) (value "MountingHole") (footprint "MountingHole:MountingHole_3.7mm")
     )
     (path "/f345e52a-8e0a-425a-b438-90809dd3b799"
-      (reference "H2") (unit 1) (value "MountingHole") (footprint "MountingHole:MountingHole_3.5mm")
+      (reference "H2") (unit 1) (value "MountingHole") (footprint "MountingHole:MountingHole_3.7mm")
     )
     (path "/bd793ae5-cde5-43f6-8def-1f95f35b1be6"
-      (reference "H3") (unit 1) (value "MountingHole") (footprint "MountingHole:MountingHole_3.5mm")
+      (reference "H3") (unit 1) (value "MountingHole") (footprint "MountingHole:MountingHole_3.7mm")
     )
     (path "/52a8f1be-73ca-41a8-bc24-2320706b0ec1"
-      (reference "H4") (unit 1) (value "MountingHole") (footprint "MountingHole:MountingHole_3.5mm")
+      (reference "H4") (unit 1) (value "MountingHole") (footprint "MountingHole:MountingHole_3.7mm")
     )
     (path "/272e9454-3a50-4c5e-bde1-b3ea68de51fa"
